Commit message: updateed bringup rviz local config and removed gazebo cmd_vel topic namespace

File: robotics_description/urdf/robot.urdf.xacro (robot description, xacro)
@@ -9,5 +9,5 @@
         align_depth="true"
         unite_imu_method="false">
-        <origin xyz="-0.1 0 0.5" rpy="0 0 0"/>
+        <origin xyz="-0.1 0 0.25" rpy="0 0 0"/>
     </xacro:sensor_d435i>
     <xacro:hokuyo_ust10_mount prefix="lidar" topic="scan" parent_link="front_mount">
