Commit message: updated robot description and simulation launch arguments

File: robotics_description/urdf/hokuyo.urdf.xacro (robot description, xacro)
@@ -2,6 +2,6 @@
 <robot xmlns:xacro="http://ros.org/wiki/xacro">
     <xacro:macro name="hokuyo" params="parent
-        name:=lidar
-        topic_ns:=lidar
+        name:=laser
+        topic_ns:=laser
         min_angle:=-1.5707963
         max_angle:=1.5707963

File: robotics_description/urdf/robot.urdf.xacro (robot description, xacro)
@@ -8,5 +8,5 @@
         align_depth="true"
         unite_imu_method="linear_interpolation">
-        <origin xyz="-0.1 0 0.25" rpy="0 0 0"/>
+        <origin xyz="-0.04 0 0.25" rpy="0 0 0"/>
     </xacro:sensor_d435i>
     <xacro:hokuyo parent="front_mount" name="hokuyo" topic_ns="hokuyo">

Commit message: added cm10a imu to replace realsense built-in one

File: robotics_description/urdf/hokuyo.urdf.xacro (robot description, xacro)
@@ -15,10 +15,10 @@
         <link name="${name}_mount">
             <visual>
-                <origin xyz="0 0 0" rpy="0 0 0" />
+                <origin xyz="0 0 0" rpy="0 0 0"/>
                 <geometry>
                     <!-- Origin of this mesh is the base of the bracket. -->
-                    <mesh filename="package://urg_node/meshes/hokuyo_ust10.stl" />
+                    <mesh filename="package://urg_node/meshes/hokuyo_ust10.stl"/>
                 </geometry>
-                <material name="dark_grey" />
+                <material name="dark_grey"/>
             </visual>
         </link>
@@ -30,7 +30,7 @@
                 <mass value="0.16" />
                 <origin xyz="0 0 0" />
-                <inertia ixx="${0.0833333 * 1.1 * (0.102 * 0.102 + 0.152 * 0.152)}" ixy="0.0" ixz="0.0"
-                    iyy="${0.0833333 * 1.1 * (0.105 * 0.105 + 0.152 * 0.152)}" iyz="0.0"
-                    izz="${0.0833333 * 1.1 * (0.105 * 0.105 + 0.102 * 0.102)}" />
+                <inertia ixx="${0.0833333 * 0.16 * (0.05 * 0.05 + 0.07 * 0.07)}" ixy="0.0" ixz="0.0"
+                    iyy="${0.0833333 * 0.16 * (0.05 * 0.05 + 0.07 * 0.07)}" iyz="0.0"
+                    izz="${0.0833333 * 0.16 * (0.05 * 0.05 + 0.05 * 0.05)}"/>
             </inertial>
         </link>

File: robotics_description/urdf/robot.urdf.xacro (robot description, xacro)
@@ -3,13 +3,16 @@
     <xacro:include filename="$(find robotics_description)/urdf/materials.urdf.xacro"/>
     <xacro:include filename="$(find robotics_description)/urdf/hokuyo.urdf.xacro"/>
+    <xacro:include filename="$(find robotics_description)/urdf/cmp10a.urdf.xacro"/>
     <xacro:include filename="$(find realsense_gazebo_description)/urdf/_d435i.urdf.xacro"/>
     <xacro:include filename="$(find scout_description)/urdf/scout_mini.urdf.xacro"/>
-    <xacro:sensor_d435i parent="front_mount" name="realsense" topics_ns="realsense"
-        align_depth="true"
-        unite_imu_method="linear_interpolation">
-        <origin xyz="-0.04 0 0.25" rpy="0 0 0"/>
-    </xacro:sensor_d435i>
     <xacro:hokuyo parent="front_mount" name="hokuyo" topic_ns="hokuyo">
         <origin xyz="-0.02 0 0" rpy="0 0 0"/>
     </xacro:hokuyo>
+    <xacro:sensor_d435i parent="front_mount" name="realsense" topics_ns="realsense"
+        align_depth="true">
+        <origin xyz="-0.04 0 0.25" rpy="0 0 0"/>
+    </xacro:sensor_d435i>
+    <xacro:cmp10a parent="front_mount" name="cmp10a" topic_ns="cmp10a">
+        <origin xyz="-0.08 0 0.25" rpy="0 0 0"/>
+    </xacro:cmp10a>
 </robot>
